File: mcu.sch (EAGLE design)
At the start: 2 parts

Commit message: experiment with different parts
Parts:
- added U$3: STM32F407VX, STM32F407Vx_LQFP100:STM32F407VX
Changed lines of the file:
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@@
 <?xml version="1.0" encoding="utf-8"?>
 <!DOCTYPE eagle SYSTEM "eagle.dtd">
-<eagle version="8.0.2">
+<eagle version="8.1.0">
 <drawing>
 <settings>
@@
 <setting verticaltext="up"/>
 </settings>
-<grid distance="0.05" unitdist="inch" unit="inch" style="lines" multiple="1" display="no" altdistance="0.01" altunitdist="inch" altunit="inch"/>
+<grid distance="0.1" unitdist="inch" unit="inch" style="lines" multiple="1" display="no" altdistance="0.01" altunitdist="inch" altunit="inch"/>
 <layers>
 <layer number="1" name="Top" color="4" fill="1" visible="no" active="no"/>
@@
 <part name="SUPPLY1" library="supply2" deviceset="VDD" device=""/>
 <part name="SUPPLY2" library="supply2" deviceset="GND" device=""/>
+<part name="U$3" library="STM32F407Vx_LQFP100" deviceset="STM32F407VX" device=""/>
 </parts>
 <sheets>
@@
 <instance part="SUPPLY1" gate="G$1" x="-168.91" y="105.41"/>
 <instance part="SUPPLY2" gate="GND" x="-116.84" y="99.06"/>
+<instance part="U$3" gate="G$1" x="53.34" y="124.46"/>
+<instance part="U$3" gate="G$2" x="53.34" y="203.2"/>
+<instance part="U$3" gate="G$3" x="124.46" y="124.46"/>
+<instance part="U$3" gate="G$4" x="124.46" y="203.2"/>
 </instances>
 <busses>
