File: ethernet_usb.sch (EAGLE design)
At the start: 11 parts, among them X1 MINI-USB_SHIELD4P-85-32004-10X, Y1 32.768kHz

Commit message: snapshot
Parts:
- added R2: 470, SparkFun-Resistors:RESISTOR0805
- added R3, R4: (no value), SparkFun-Resistors:RESISTOR0805
Connections:
- new net 3.3V: U1.VCCIOA, U1.VCCIOB
- new net 5V: R2.2, U1.VCC0, U1.VCC1
- new net N$12: R2.1, R3.2, U1.AVVC
- new net N$16: R4.2, U1.3V3OUT
- net GND: now also R3.1, R4.1, U1.AGND, U1.GND0, U1.GND1, U1.GND2, U1.GND3
Other:
- note added: "100nF CAP"
- note added: "33nF CAP"
Changed lines of the file:
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@@
 <part name="C3" library="SparkFun-Capacitors" deviceset="1.0UF" device="-0805-25V-10%" value="1.0uF"/>
 <part name="C4" library="SparkFun-Capacitors" deviceset="1.0UF" device="-0805-25V-10%" value="1.0uF"/>
+<part name="GND4" library="SparkFun-PowerSymbols" deviceset="GND" device=""/>
+<part name="SUPPLY1" library="SparkFun-PowerSymbols" deviceset="5V" device=""/>
+<part name="SUPPLY3" library="SparkFun-PowerSymbols" deviceset="3.3V" device=""/>
+<part name="R2" library="SparkFun-Resistors" deviceset="RESISTOR" device="0805" value=" 470"/>
+<part name="R3" library="SparkFun-Resistors" deviceset="RESISTOR" device="0805" value=" "/>
+<part name="GND5" library="SparkFun-PowerSymbols" deviceset="GND" device=""/>
+<part name="R4" library="SparkFun-Resistors" deviceset="RESISTOR" device="0805" value=" "/>
 </parts>
 <sheets>
 <sheet>
 <plain>
+<text x="-584.2" y="436.88" size="1.778" layer="91">33nF CAP</text>
+<text x="-581.66" y="454.66" size="1.778" layer="91">100nF CAP</text>
 </plain>
 <instances>
@@
 <instance part="C3" gate="G$1" x="-627.38" y="259.08"/>
 <instance part="C4" gate="G$1" x="-617.22" y="259.08"/>
+<instance part="GND4" gate="1" x="-541.02" y="350.52"/>
+<instance part="SUPPLY1" gate="G$1" x="-548.64" y="467.36"/>
+<instance part="SUPPLY3" gate="G$1" x="-541.02" y="467.36"/>
+<instance part="R2" gate="G$1" x="-553.72" y="457.2" rot="R90"/>
+<instance part="R3" gate="G$1" x="-571.5" y="449.58"/>
+<instance part="GND5" gate="1" x="-589.28" y="426.72"/>
+<instance part="R4" gate="G$1" x="-579.12" y="431.8"/>
 </instances>
 <busses>
@@
 <wire x1="-622.3" y1="251.46" x2="-622.3" y2="254" width="0.1524" layer="91"/>
 <junction x="-622.3" y="254"/>
+</segment>
+<segment>
+<pinref part="U1" gate="G$1" pin="AGND"/>
+<wire x1="-553.72" y1="358.14" x2="-553.72" y2="355.6" width="0.1524" layer="91"/>
+<pinref part="GND4" gate="1" pin="GND"/>
+<wire x1="-553.72" y1="355.6" x2="-548.64" y2="355.6" width="0.1524" layer="91"/>
+<wire x1="-548.64" y1="355.6" x2="-546.1" y2="355.6" width="0.1524" layer="91"/>
+<wire x1="-546.1" y1="355.6" x2="-543.56" y2="355.6" width="0.1524" layer="91"/>
+<wire x1="-543.56" y1="355.6" x2="-541.02" y2="355.6" width="0.1524" layer="91"/>
+<wire x1="-541.02" y1="355.6" x2="-541.02" y2="353.06" width="0.1524" layer="91"/>
+<pinref part="U1" gate="G$1" pin="GND0"/>
+<wire x1="-541.02" y1="358.14" x2="-541.02" y2="355.6" width="0.1524" layer="91"/>
+<junction x="-541.02" y="355.6"/>
+<pinref part="U1" gate="G$1" pin="GND1"/>
+<wire x1="-543.56" y1="358.14" x2="-543.56" y2="355.6" width="0.1524" layer="91"/>
+<junction x="-543.56" y="355.6"/>
+<pinref part="U1" gate="G$1" pin="GND2"/>
+<wire x1="-546.1" y1="358.14" x2="-546.1" y2="355.6" width="0.1524" layer="91"/>
+<junction x="-546.1" y="355.6"/>
+<pinref part="U1" gate="G$1" pin="GND3"/>
+<wire x1="-548.64" y1="358.14" x2="-548.64" y2="355.6" width="0.1524" layer="91"/>
+<junction x="-548.64" y="355.6"/>
+</segment>
+<segment>
+<pinref part="GND5" gate="1" pin="GND"/>
+<wire x1="-589.28" y1="429.26" x2="-589.28" y2="431.8" width="0.1524" layer="91"/>
+<pinref part="R3" gate="G$1" pin="1"/>
+<wire x1="-589.28" y1="431.8" x2="-589.28" y2="449.58" width="0.1524" layer="91"/>
+<wire x1="-589.28" y1="449.58" x2="-576.58" y2="449.58" width="0.1524" layer="91"/>
+<pinref part="R4" gate="G$1" pin="1"/>
+<wire x1="-584.2" y1="431.8" x2="-589.28" y2="431.8" width="0.1524" layer="91"/>
+<junction x="-589.28" y="431.8"/>
 </segment>
 </net>
@@
 </segment>
 </net>
+<net name="N$12" class="0">
+<segment>
+<pinref part="R3" gate="G$1" pin="2"/>
+<wire x1="-566.42" y1="449.58" x2="-553.72" y2="449.58" width="0.1524" layer="91"/>
+<pinref part="R2" gate="G$1" pin="1"/>
+<wire x1="-553.72" y1="449.58" x2="-553.72" y2="452.12" width="0.1524" layer="91"/>
+<pinref part="U1" gate="G$1" pin="AVVC"/>
+<wire x1="-553.72" y1="447.04" x2="-553.72" y2="449.58" width="0.1524" layer="91"/>
+<junction x="-553.72" y="449.58"/>
+</segment>
+</net>
+<net name="5V" class="0">
+<segment>
+<pinref part="SUPPLY1" gate="G$1" pin="5V"/>
+<pinref part="U1" gate="G$1" pin="VCC0"/>
+<wire x1="-548.64" y1="467.36" x2="-548.64" y2="464.82" width="0.1524" layer="91"/>
+<pinref part="R2" gate="G$1" pin="2"/>
+<wire x1="-548.64" y1="464.82" x2="-548.64" y2="447.04" width="0.1524" layer="91"/>
+<wire x1="-553.72" y1="462.28" x2="-553.72" y2="464.82" width="0.1524" layer="91"/>
+<wire x1="-553.72" y1="464.82" x2="-548.64" y2="464.82" width="0.1524" layer="91"/>
+<junction x="-548.64" y="464.82"/>
+<pinref part="U1" gate="G$1" pin="VCC1"/>
+<wire x1="-546.1" y1="447.04" x2="-546.1" y2="464.82" width="0.1524" layer="91"/>
+<wire x1="-546.1" y1="464.82" x2="-548.64" y2="464.82" width="0.1524" layer="91"/>
+</segment>
+</net>
+<net name="3.3V" class="0">
+<segment>
+<pinref part="SUPPLY3" gate="G$1" pin="3.3V"/>
+<pinref part="U1" gate="G$1" pin="VCCIOB"/>
+<wire x1="-541.02" y1="467.36" x2="-541.02" y2="464.82" width="0.1524" layer="91"/>
+<pinref part="U1" gate="G$1" pin="VCCIOA"/>
+<wire x1="-541.02" y1="464.82" x2="-541.02" y2="447.04" width="0.1524" layer="91"/>
+<wire x1="-543.56" y1="447.04" x2="-543.56" y2="464.82" width="0.1524" layer="91"/>
+<wire x1="-543.56" y1="464.82" x2="-541.02" y2="464.82" width="0.1524" layer="91"/>
+<junction x="-541.02" y="464.82"/>
+</segment>
+</net>
+<net name="N$16" class="0">
+<segment>
+<pinref part="U1" gate="G$1" pin="3V3OUT"/>
+<pinref part="R4" gate="G$1" pin="2"/>
+<wire x1="-571.5" y1="431.8" x2="-574.04" y2="431.8" width="0.1524" layer="91"/>
+</segment>
+</net>
